File: EAGLE Models/sbRIO Daughter Card v5/Daughter Card Schematic v5.brd (EAGLE design)
At the start: 101.6 x 81.3 mm, 110 parts, among them Q1 MMBT4403-7-F, Q10 MMBT4403-7-F, Q11 MMBT4401-7-F, Q13 MMBT4401-7-F, Q14 MMBT4403-7-F, Q15 MMBT4403-7-F, Q16 MMBT4403-7-F, Q17 MMBT4403-7-F, Q2 MMBT4403-7-F, Q3 MMBT4403-7-F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

Commit message: made many changes
Parts:
- removed DASHBOARD_CONN, HV_BOX_CONN, PEDAL_CONN, SHOCK_POT_CONN, WHEEL_SPEED: EN3_PCB_8, formula electric:EN3_PCB_8
- removed Q14, Q15, Q16, Q17: MMBT4403-7-F, formula electric:SOT-23-3
- removed R26, R28, R30, R32: 10k, resistor:R0402
- removed R27, R29, R31, R33: 1k, resistor:R0402
- added ACCUMULATOR_CONN: RJ45-6L21-S, con-tycoelectronics:RJ45-SHIELD1
- added AIO_PO_CONN, TUB_CONN: 2516-5, con-3m:PAK100/2500-5-16
- added F19, F20, F21, F22, F23, F24, F25, F26: (no value), resistor:R0402
- added Q12, Q18, Q19, Q20: MMBT4403-7-F, formula electric:SOT-23-3
- added R37, R38, R39, R40, R41, R42, R43, R44: 4.7k, resistor:R0402
- added U$1, U$4, U$5, U$6: MMBT4401-7-F, formula electric:SOT-23-3
- moved F15 228.4 mm to (-1.52, -147.6), flipped to the top, turned to 0 degrees
- moved F10 85.0 mm to (7.49, 57.5), flipped to the bottom, turned to 0 degrees
- moved F16 84.9 mm to (4.83, 58.3), flipped to the bottom, turned to 0 degrees
- moved F9 73.7 mm to (7.49, 59.2), flipped to the bottom, turned to 0 degrees
- moved D3 55.8 mm to (61.2, 45.9)
- moved F11 48.6 mm to (44.1, 55.2), flipped to the top
- moved F12 48.6 mm to (44.1, 51.4), flipped to the top
- moved F13 48.6 mm to (44.1, 47.6), flipped to the top
- moved F14 48.6 mm to (44.1, 43.8), flipped to the top
- moved Q3 43.6 mm to (46.6, 48.3), flipped to the top
- moved Q4 43.6 mm to (46.6, 44.5), flipped to the top
- moved Q5 43.6 mm to (46.6, 52.1), flipped to the top
- moved Q6 43.6 mm to (46.6, 55.9), flipped to the top
- moved C10 38.6 mm to (44.2, 58.2)
- moved R19 38.6 mm to (49.0, 48.0), flipped to the top
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Connections:
- removed net N$84: Q17.P$2, R32.2
- new net DIO25: R41.1
- new net DIO26: R37.2
- new net DIO27: R38.2
- new net DIO28: R39.2
- new net N$29: AIO_PO_CONN.3, F19.2
- new net N$30: Q19.P$2, R40.2
- new net N$31: R40.1, U$1.P$1
- new net N$32: R41.2, U$1.P$2
- new net N$85: Q12.P$2, R42.2
- new net N$86: R42.1, U$4.P$1
- new net N$87: R37.1, U$4.P$2
- new net N$88: Q18.P$2, R43.2
- new net N$89: R43.1, U$5.P$1
- new net N$90: R38.1, U$5.P$2
- new net N$91: Q20.P$2, R44.2
- new net N$92: R44.1, U$6.P$1
- new net N$93: R39.1, U$6.P$2
- new net PO1: F26.1, Q19.P$1
- new net PO2: F25.1, Q12.P$1
- new net PO3: F24.1, Q18.P$1
- new net PO4: F23.1, Q20.P$1
- net 12V: now also F19.1, Q12.P$3, Q18.P$3, Q19.P$3, Q20.P$3; no longer F15.2
- net 3.3V: no longer Q14.P$3, Q15.P$3, Q16.P$3, Q17.P$3
- net AI1: now also ACCUMULATOR_CONN.5; no longer HV_BOX_CONN.P$5
- net AI10: now also AIO_PO_CONN.5; no longer SHOCK_POT_CONN.P$2
- net AI11: now also AIO_PO_CONN.4; no longer SHOCK_POT_CONN.P$3
- net AI15: now also AIO_PO_CONN.8
- net AI2: now also ACCUMULATOR_CONN.6; no longer HV_BOX_CONN.P$6
- net AI3: now also TUB_CONN.10; no longer PEDAL_CONN.P$7
- net AI4: now also TUB_CONN.9; no longer PEDAL_CONN.P$8
- net AI7: now also TUB_CONN.13; no longer PEDAL_CONN.P$4
- net AI8: now also AIO_PO_CONN.7; no longer SHOCK_POT_CONN.P$8
- net AI9: now also AIO_PO_CONN.6; no longer SHOCK_POT_CONN.P$1
- net AO0: now also F22.1
- net AO1: now also F21.1
- net AO2: now also F20.1
- net AO3: now also F15.1
- net CAN_GND: now also ACCUMULATOR_CONN.1, ACCUMULATOR_CONN.S1, ACCUMULATOR_CONN.S2, ACCUMULATOR_CONN.S3, ACCUMULATOR_CONN.S4; no longer HV_BOX_CONN.P$1
- net CAN_H: now also ACCUMULATOR_CONN.3, TUB_CONN.7; no longer DASHBOARD_CONN.P$2, HV_BOX_CONN.P$3
- net CAN_L: now also ACCUMULATOR_CONN.4, TUB_CONN.6; no longer DASHBOARD_CONN.P$3, HV_BOX_CONN.P$4
- net DI09: now also TUB_CONN.8; no longer DASHBOARD_CONN.P$1
- net DIO0: no longer Q14.P$1, R27.2
- net DIO1: no longer Q17.P$1, R33.2
- net DIO2: no longer Q16.P$1, R31.2
- net DIO3: no longer Q15.P$1, R29.2
- net GND: now also AIO_PO_CONN.1, TUB_CONN.11, U$1.P$3, U$4.P$3, U$5.P$3, U$6.P$3; no longer R27.1, R29.1, R31.1, R33.1, SHOCK_POT_CONN.P$7, WHEEL_SPEED.P$5
- net N$10: now also AIO_PO_CONN.12, F22.2; no longer R26.1, WHEEL_SPEED.P$8
- net N$13: now also ACCUMULATOR_CONN.7; no longer HV_BOX_CONN.P$7
- net N$14: now also ACCUMULATOR_CONN.8; no longer HV_BOX_CONN.P$8
- net N$20: now also AIO_PO_CONN.2; no longer SHOCK_POT_CONN.P$4
- net N$21: now also AIO_PO_CONN.13, F23.2; no longer F15.1, WHEEL_SPEED.P$4
- net N$22: now also TUB_CONN.12; no longer PEDAL_CONN.P$5
- net N$23: now also TUB_CONN.5; no longer DASHBOARD_CONN.P$4
- net N$24: now also TUB_CONN.4; no longer DASHBOARD_CONN.P$5
- net N$3: now also AIO_PO_CONN.9, F15.2; no longer R32.1, WHEEL_SPEED.P$1
- net N$33: now also TUB_CONN.3; no longer DASHBOARD_CONN.P$6
- net N$34: now also TUB_CONN.2; no longer DASHBOARD_CONN.P$7
- net N$35: now also TUB_CONN.1; no longer DASHBOARD_CONN.P$8
- net N$6: now also AIO_PO_CONN.10, F20.2; no longer Q16.P$2, R30.2
- net N$81: now also AIO_PO_CONN.14, F24.2; no longer Q14.P$2, R26.2
- net N$82: now also AIO_PO_CONN.15, F25.2; no longer Q15.P$2, R28.2
- net N$83: now also AIO_PO_CONN.16, F26.2; no longer R30.1, WHEEL_SPEED.P$2
- net N$9: now also AIO_PO_CONN.11, F21.2; no longer R28.1, WHEEL_SPEED.P$3
- net SHIELD: now also ACCUMULATOR_CONN.2; no longer HV_BOX_CONN.P$2
- net STEERING_POS: now also TUB_CONN.14; no longer PEDAL_CONN.P$3
- net THROTTLE_1: now also TUB_CONN.16; no longer PEDAL_CONN.P$1
- net THROTTLE_2: now also TUB_CONN.15; no longer PEDAL_CONN.P$2
Routing:
- net 5V: track 166.1 -> 10.2 mm
- net 3.3V: track 211.1 -> 84.2 mm, vias 5 -> 4
- net CAN_H: track 138.2 -> 13.1 mm
- net CAN_L: track 150.8 -> 43.9 mm
- net GND: track 648.3 -> 565.0 mm, vias 6 -> 7
- net N$15: track 78.3 -> 22.5 mm
- net DIO14: track 50.6 -> 0.00 mm, vias 3 -> 0
- net N$18: track 47.9 -> 0.00 mm, vias 2 -> 0
- net N$16: track 69.7 -> 23.2 mm
- net N$17: track 44.9 -> 0.00 mm, vias 1 -> 0
- net 12V: track 232.8 -> 191.6 mm, vias 5 -> 6
- net AI1: track 38.7 -> 0.00 mm, vias 1 -> 0
- net AI2: track 90.8 -> 54.8 mm, vias 1 -> 0
- net DIO1: track 35.1 -> 0.00 mm, vias 2 -> 0
- net N$4: track 81.1 -> 47.2 mm, vias 2 -> 0
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- removed copper zone on layer 16, net 12V

Commit message: Changed daughter card stuff
Parts:
- removed Q12, Q18, Q19, Q20: MMBT4403-7-F, formula electric:SOT-23-3
- removed R37, R38, R39, R40, R41, R42, R43, R44: 4.7k, resistor:R0402
- removed U$1, U$4, U$5, U$6: MMBT4401-7-F, formula electric:SOT-23-3
- added IC1: ITS4880R-PAD, infineon:PG-DSO-36PAD
- moved D6 0.57 mm to (46.5, 11.8)
Connections:
- removed net DIO25: R41.1
- removed net DIO26: R37.2
- removed net N$30: Q19.P$2, R40.2
- removed net N$87: R37.1, U$4.P$2
- removed net N$88: Q18.P$2, R43.2
- removed net N$89: R43.1, U$5.P$1
- removed net N$90: R38.1, U$5.P$2
- removed net N$91: Q20.P$2, R44.2
- removed net N$92: R44.1, U$6.P$1
- removed net N$93: R39.1, U$6.P$2
- net 12V: now also IC1.3, IC1.TH@1, IC1.TH@2; no longer Q12.P$3, Q18.P$3, Q19.P$3, Q20.P$3
- net DIO27: now also IC1.8; no longer R38.2
- net DIO28: now also IC1.9; no longer R39.2
- net GND: now also IC1.19; no longer U$1.P$3, U$4.P$3, U$5.P$3, U$6.P$3
- net N$31: now also IC1.27, IC1.28; no longer R40.1, U$1.P$1
- net N$32: now also IC1.25, IC1.26; no longer R41.2, U$1.P$2
- net N$85: now also IC1.23, IC1.24; no longer Q12.P$2, R42.2
- net N$86: now also IC1.21, IC1.22; no longer R42.1, U$4.P$1
- net PO1: now also IC1.35, IC1.36; no longer Q19.P$1
- net PO2: now also IC1.33, IC1.34; no longer Q12.P$1
- net PO3: now also IC1.31, IC1.32; no longer Q18.P$1
- net PO4: now also IC1.29, IC1.30; no longer Q20.P$1

Commit message: stuff
Parts:
- removed F11, F12, F13, F14, F23, F24, F25, F26: (no value), resistor:R0402
- removed Q3, Q4, Q5, Q6: MMBT4403-7-F, formula electric:SOT-23-3
- removed R10, R18, R19, R20, R21, R5, R6, R7: 4.7k, resistor:R0402
- removed U$17, U$18, U$19, U$20: MMBT4401-7-F, formula electric:SOT-23-3
- moved TUB_CONN 211.5 mm to (8.26, 35.6), turned to 90 degrees
- moved IC1 204.4 mm to (65.2, 7.75)
- moved F22 198.9 mm to (36.6, 40.8), flipped to the bottom, turned to 90 degrees
- moved F21 196.3 mm to (34.5, 40.8), flipped to the bottom, turned to 90 degrees
- moved F20 193.6 mm to (32.3, 40.8), flipped to the bottom, turned to 90 degrees
- moved F15 191.0 mm to (30.0, 40.8), flipped to the bottom, turned to 90 degrees
- moved F19 19.8 mm to (12.6, 71.1)
- moved F10 19.8 mm to (10.8, 77.1)
- moved F16 19.8 mm to (8.13, 77.9)
- moved AIO_PO_CONN 19.8 mm to (8.51, 64.8)
- moved F9 19.8 mm to (10.8, 78.7)
Connections:
- removed net N$21: AIO_PO_CONN.13, F23.2
- removed net N$24: F11.1, TUB_CONN.4
- removed net N$31: IC1.27, IC1.28
- removed net N$32: IC1.25, IC1.26
- removed net N$33: F12.1, TUB_CONN.3
- removed net N$34: F13.1, TUB_CONN.2
- removed net N$35: F14.1, TUB_CONN.1
- removed net N$5: Q6.P$2, R21.2
- removed net N$50: Q5.P$2, R5.2
- removed net N$51: Q3.P$2, R19.2
- removed net N$64: R5.1, U$17.P$1
- removed net N$65: R18.2, U$17.P$2
- removed net N$66: R19.1, U$18.P$1
- removed net N$67: R6.1, U$18.P$2
- removed net N$68: Q4.P$2, R20.2
- removed net N$69: R20.1, U$19.P$1
- removed net N$70: R7.1, U$19.P$2
- removed net N$71: R21.1, U$20.P$1
- removed net N$72: R10.1, U$20.P$2
- removed net N$82: AIO_PO_CONN.15, F25.2
- removed net N$85: IC1.23, IC1.24
- removed net N$86: IC1.21, IC1.22
- new net DIO25: IC1.6
- new net DIO26: IC1.7
- net 12V: no longer Q3.P$3, Q4.P$3, Q5.P$3, Q6.P$3
- net AMS_OUT: now also IC1.27, IC1.28; no longer F12.2, Q5.P$1
- net BSPD_OUT: now also IC1.23, IC1.24; no longer F14.2, Q4.P$1
- net BUZZER_OUT: now also IC1.21, IC1.22; no longer F11.2, Q6.P$1
- net DIO14: now also IC1.13; no longer R10.2
- net DIO6: now also IC1.10; no longer R18.1
- net DIO7: now also IC1.11; no longer R6.2
- net DIO8: now also IC1.12; no longer R7.2
- net GND: no longer U$17.P$3, U$18.P$3, U$19.P$3, U$20.P$3
- net IMD_OUT: now also IC1.25, IC1.26; no longer F13.2, Q3.P$1
- net N$81: no longer F24.2
- net N$83: no longer F26.2
- net PO1: no longer F26.1
- net PO2: no longer F25.1
- net PO3: no longer F24.1
- net PO4: no longer F23.1
Routing:
- net GND: track 565.0 -> 514.7 mm, vias 7 -> 8
- net CAN_H: track 13.1 -> 50.3 mm, vias 0 -> 1
- net 12V: track 191.6 -> 166.8 mm
- net DIO7: track 42.7 -> 40.3 mm
- net N$66: track 1.67 -> 0.00 mm
- net N$68: track 1.56 -> 0.00 mm
- net N$5: track 1.56 -> 0.00 mm
- net N$71: track 1.55 -> 0.00 mm
- net N$64: track 1.55 -> 0.00 mm
- net IMD_OUT: track 1.55 -> 0.00 mm
- net BUZZER_OUT: track 1.55 -> 0.00 mm
- net BSPD_OUT: track 1.55 -> 0.00 mm
- net AMS_OUT: track 1.55 -> 0.00 mm
- net N$69: track 1.55 -> 0.00 mm
- net N$50: track 1.54 -> 0.00 mm
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
Commit message: Committed daughter card before autorouting
Parts:
- moved IC1 47.1 mm to (37.2, 45.7), flipped to the bottom, turned to 270 degrees
- moved D3 36.3 mm to (83.1, 17.0)
- moved D2 11.5 mm to (88.8, 28.6)
- moved R14 10.4 mm to (86.6, 23.7), turned to 270 degrees
- moved F22 9.83 mm to (31.2, 32.5)
- moved F21 9.63 mm to (29.6, 32.5)
- moved R13 8.32 mm to (82.7, 11.4)
- moved D5 8.13 mm to (38.1, 3.94)
- moved D6 8.13 mm to (46.6, 3.68)
- moved F17 8.13 mm to (83.8, 21.6)
- moved F7 8.13 mm to (40.3, 2.16)
- moved F8 8.13 mm to (43.9, 2.16)
- moved Q7 8.13 mm to (81.3, 20.4)
- moved R11 8.13 mm to (80.3, 17.3)
- moved R16 8.13 mm to (76.7, 20.2)
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Connections:
- net N$17 renamed DIO23
- net N$18 renamed DIO24
- removed net N$25: U$3.153
- removed net N$26: U$3.141
- removed net N$27: U$3.135
- removed net N$28: U$3.123
- removed net N$81: AIO_PO_CONN.14
- removed net N$83: AIO_PO_CONN.16
- new net N$21: IC1.TH@11
- new net N$5: IC1.TH@6, IC1.TH@7
- net 12V: now also IC1.TH@12
- net DIO25: now also U$3.153
- net DIO26: now also U$3.141
- net DIO27: now also U$3.135
- net DIO28: now also U$3.123
- net PO1: now also AIO_PO_CONN.16
- net PO2: now also AIO_PO_CONN.15
- net PO3: now also AIO_PO_CONN.14
- net PO4: now also AIO_PO_CONN.13
Routing:
- net 12V: track 166.8 -> 244.5 mm
- net GND: track 514.7 -> 555.1 mm
- net N$4: track 47.2 -> 7.36 mm, vias 0 -> 1
- net N$5: track 0.00 -> 16.2 mm
- net DIO14: track 0.00 -> 15.9 mm
- net N$2: track 44.5 -> 56.1 mm, vias 0 -> 1
- net DIO13: track 41.7 -> 32.6 mm
- net N$1: track 16.1 -> 7.90 mm
- net AI2: track 54.8 -> 62.9 mm
- net DIO16: track 59.9 -> 68.0 mm
- net DIO17: track 39.5 -> 47.7 mm
- net AI3: track 54.8 -> 62.9 mm
- net DIO18: track 35.3 -> 43.4 mm
- net DIO19: track 41.1 -> 49.2 mm
- net DIO38: track 25.6 -> 33.7 mm
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
Commit message: fixed more traces
Parts:
- moved R36 18.5 mm to (67.4, 52.1)
- moved F20 11.9 mm to (31.1, 33.0)
- moved F15 11.8 mm to (28.8, 33.1)
- moved F22 4.74 mm to (35.9, 33.1)
- moved F21 3.99 mm to (33.5, 33.1)
- moved TUB_CONN 0.57 mm to (8.51, 36.1), flipped to the bottom, turned to 270 degrees
Routing:
- net DIO9: track 48.5 -> 24.1 mm
- net DIO6: track 40.2 -> 56.6 mm
- net DIO7: track 40.3 -> 55.9 mm
- net GND: track 555.1 -> 541.9 mm, vias 8 -> 9
- net DIO8: track 45.4 -> 57.4 mm
- net CAN_L: track 42.8 -> 52.8 mm, vias 0 -> 1
- net 12V: track 244.5 -> 235.7 mm, vias 6 -> 5
- net AO3: track 21.9 -> 29.1 mm
- net AO2: track 21.9 -> 28.9 mm
- net AO1: track 21.9 -> 28.8 mm
- net AO0: track 21.9 -> 28.8 mm
- net CAN_H: track 50.3 -> 51.1 mm, vias 1 -> 2

Commit message: fixed four outputs not connected in schematic
Connections:
- net AMS_OUT: now also TUB_CONN.3
- net BSPD_OUT: now also TUB_CONN.1
- net BUZZER_OUT: now also TUB_CONN.4
- net IMD_OUT: now also TUB_CONN.2
Changed lines of the file:
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@@
 <contactref element="IC1" pad="28"/>
 <contactref element="IC1" pad="27"/>
-<wire x1="30.711" y1="46.045" x2="30.711" y2="45.395" width="0" layer="19" extent="1-1"/>
+<contactref element="TUB_CONN" pad="3"/>
+<wire x1="30.711" y1="45.395" x2="30.711" y2="46.045" width="0" layer="19" extent="16-16"/>
+<wire x1="9.779" y1="42.418" x2="30.711" y2="45.395" width="0" layer="19" extent="16-16"/>
 </signal>
 <signal name="IMD_OUT">
 <contactref element="IC1" pad="26"/>
 <contactref element="IC1" pad="25"/>
-<wire x1="30.711" y1="44.095" x2="30.711" y2="44.745" width="0" layer="19" extent="1-1"/>
+<contactref element="TUB_CONN" pad="2"/>
+<wire x1="30.711" y1="44.095" x2="30.711" y2="44.745" width="0" layer="19" extent="16-16"/>
+<wire x1="7.239" y1="44.958" x2="30.711" y2="44.745" width="0" layer="19" extent="16-16"/>
 </signal>
 <signal name="BSPD_OUT">
 <contactref element="IC1" pad="24"/>
 <contactref element="IC1" pad="23"/>
-<wire x1="30.711" y1="43.445" x2="30.711" y2="42.795" width="0" layer="19" extent="1-1"/>
+<contactref element="TUB_CONN" pad="1"/>
+<wire x1="30.711" y1="42.795" x2="30.711" y2="43.445" width="0" layer="19" extent="16-16"/>
+<wire x1="9.779" y1="44.958" x2="30.711" y2="43.445" width="0" layer="19" extent="16-16"/>
 </signal>
 <signal name="BUZZER_OUT">
 <contactref element="IC1" pad="22"/>
 <contactref element="IC1" pad="21"/>
-<wire x1="30.711" y1="41.495" x2="30.711" y2="42.145" width="0" layer="19" extent="1-1"/>
+<contactref element="TUB_CONN" pad="4"/>
+<wire x1="30.711" y1="41.495" x2="30.711" y2="42.145" width="0" layer="19" extent="16-16"/>
+<wire x1="7.239" y1="42.418" x2="30.711" y2="42.145" width="0" layer="19" extent="16-16"/>
 </signal>
 <signal name="PO1">

Commit message: did more things
Parts:
- moved F7 10.4 mm to (31.1, 7.11), flipped to the top
- moved F8 5.85 mm to (39.1, 5.46), flipped to the top, turned to 90 degrees
- moved D6 5.68 mm to (41.5, 6.22), flipped to the top, turned to 90 degrees
- moved D5 4.94 mm to (33.7, 6.10), flipped to the top, turned to 90 degrees
- moved R9 0.80 mm to (44.3, 6.22), flipped to the top, turned to 90 degrees
- moved R8 0.18 mm to (36.7, 7.11), flipped to the top, turned to 0 degrees
Routing:
- net AI1: track 0.00 -> 80.1 mm, vias 0 -> 2
- net AI2: track 62.9 -> 132.3 mm, vias 0 -> 2
- net N$15: track 21.3 -> 66.4 mm, vias 1 -> 0
- net N$16: track 19.2 -> 58.2 mm, vias 1 -> 0
- net CAN_GND: track 48.1 -> 57.9 mm
- net GND: track 541.9 -> 548.5 mm, vias 9 -> 11
- net AMS_OK: track 2.12 -> 0.00 mm
- net IMD_OK: track 1.83 -> 0.00 mm
