File: EAGLE Models/sbRIO Daughter Card v5/Daughter Card Schematic v5.sch (EAGLE design)
At the start: 81 parts, among them IC1 ITS4880R-PAD, Q1 MMBT4403-7-F, Q10 MMBT4403-7-F, Q11 MMBT4401-7-F, Q13 MMBT4401-7-F, Q2 MMBT4403-7-F, Q7 MMBT4403-7-F, Q8 MMBT4403-7-F, Q9 MMBT4401-7-F, U1 MMBT4403-7-F, U2 ADXL345, U3 L3G4200D

Commit message: made daughter card amplifiers all based off of  ICs
Parts:
- removed F: (no value), resistor:R-EU_R0402
- removed Q1, Q10, Q2, U1: MMBT4403-7-F, formula electric:MMBT4403-7-F
- removed Q11, Q13, Q9, U$23: MMBT4401-7-F, formula electric:MMBT4401-7-F
- removed R1, R2, R23, R24, R25, R3: 5k, resistor:R-US_R0402
- removed R22, R4: 4.7k, resistor:R-US_R0402
- added F14: (no value), resistor:R-EU_R0402
- added IC2, IC3: BTS716G, infineon:BTS716G
- IC1: value ITS4880R-PAD -> BTS716G; device infineon:ITS4880R-PAD -> infineon:BTS716G
Connections:
- net DI09 renamed DI02
- removed net N$16: D6.A, R9.1, U$3.DIO5
- removed net N$21: IC1P1.VBB@9
- removed net N$36: F.2, SHTDWN_CONN.4
- removed net N$39: F1.2, SHTDWN_CONN.2
- removed net N$40: F2.2, SHTDWN_CONN.1
- removed net N$44: F.1, U1.C
- removed net N$45: F6.2, Q10.C
- removed net N$46: R23.2, U1.B
- removed net N$47: Q1.B, R2.2
- removed net N$48: Q2.B, R3.2
- removed net N$49: Q10.B, R22.2
- removed net N$7: F1.1, Q1.C
- removed net N$73: Q9.C, R22.1
- removed net N$74: Q9.B, R4.2
- removed net N$75: Q13.C, R23.1
- removed net N$76: Q13.B, R1.2
- removed net N$77: R2.1, U$23.C
- removed net N$78: Q11.C, R3.1
- removed net N$79: R24.2, U$23.B
- removed net N$8: F2.1, Q2.C
- removed net N$80: Q11.B, R25.2
- new net BSPD5: F6.2, IC2G$1.OUT1
- new net DIO21: IC2G$1.IN2, U$3.DIO21
- new net DIO22: IC2G$1.IN3, U$3.DIO22
- new net DIO4: U$3.DIO4
- new net DIO44: R16.1, U$3.DIO44
- new net DIO45: R15.1, U$3.DIO45
- new net DIO48: U$3.DIO48, U2.INT1
- new net DIO5: U$3.DIO5
- new net DIO81: U$3.DIO81, U2.SDO, U3.SDO
- new net DIO82: U$3.DIO82
- new net DIO83: U$3.DIO83
- new net DIO85: U$3.DIO85
- new net DIO86: U$3.DIO86
- new net DIO87: U$3.DIO87
- new net DIO90: IC3G$1.IN3, U$3.DIO90
- new net DIO91: IC3G$1.IN4, U$3.DIO91
- new net DIO92: IC3G$1.IN1, U$3.DIO92
- new net DIO93: IC3G$1.IN2, U$3.DIO93
- new net DIO94: D5.A, R8.2, U$3.DIO94
- new net DIO95: D6.A, R9.1, U$3.DIO95
- new net N$24: U$3.DIO88
- new net SHUTDOWN_1: F14.1, IC2G$1.OUT2
- new net SHUTDOWN_2: F2.1, IC2G$1.OUT3
- new net SHUTDOWN_3: F1.1, IC2G$1.OUT4
- net 12V: now also IC1G$2.VBB@1, IC1G$2.VBB@2, IC1G$2.VBB@3, IC1G$2.VBB@4, IC1G$2.VBB@5, IC1G$2.VBB@6, IC1G$2.VBB@7, IC1G$2.VBB@8, IC2G$2.VBB@1, IC2G$2.VBB@2, IC2G$2.VBB@3, IC2G$2.VBB@4, IC2G$2.VBB@5, IC2G$2.VBB@6, IC2G$2.VBB@7, IC2G$2.VBB@8, IC3G$2.VBB@1, IC3G$2.VBB@2, IC3G$2.VBB@3, IC3G$2.VBB@4, IC3G$2.VBB@5, IC3G$2.VBB@6, IC3G$2.VBB@7, IC3G$2.VBB@8, SHTDWN_CONN.4; no longer IC1''.LS, IC1''.VBB, IC1''.VBB@1, IC1P1.VBB@10, Q1.E, Q10.E, Q2.E, SHTDWN_CONN.3, U1.E
- net AMS_OUT: now also IC3G$1.OUT2; no longer IC1''.OUT5, IC1''.OUT5@2
- net BSPD_OUT: now also IC3G$1.OUT4; no longer IC1''.OUT7, IC1''.OUT7@2
- net BUZZER_OUT: now also IC3G$1.OUT1; no longer IC1''.OUT8, IC1''.OUT8@2
- net DIO1: now also D4.A, R34.2
- net DIO10: no longer D4.A, R34.2
- net DIO11: no longer R1.1
- net DIO12: no longer D2.A, R14.1
- net DIO13: now also D1.A, R17.1; no longer R4.1
- net DIO14: now also D2.A, R14.1; no longer IC1''.IN8, SBRIO_AUX.DIO14
- net DIO15: no longer SBRIO_AUX.DIO15
- net DIO16: now also U2.CS; no longer R16.1, SBRIO_AUX.DIO16
- net DIO17: now also U2.INT2; no longer SBRIO_AUX.DIO17
- net DIO18: now also U2.SDA, U3.SDA/SDI; no longer SBRIO_AUX.DIO18
- net DIO19: no longer SBRIO_AUX.DIO19
- net DIO2: now also R36.2
- net DIO20: no longer D1.A, R17.1
- net DIO25: now also IC1G$1.IN1; no longer IC1''.IN1
- net DIO26: now also IC1G$1.IN2; no longer IC1''.IN2
- net DIO27: now also IC1G$1.IN3; no longer IC1''.IN3
- net DIO28: now also IC1G$1.IN4; no longer IC1''.IN4
- net DIO29: no longer U2.CS
- net DIO30: no longer U2.SDO, U3.SDO
- net DIO31: no longer U2.SDA, U3.SDA/SDI
- net DIO36: no longer U2.INT1
- net DIO37: no longer U2.INT2
- net DIO38: no longer SBRIO_AUX.DIO38
- net DIO39: no longer R15.1
- net DIO6: now also IC2G$1.IN1; no longer IC1''.IN5
- net DIO7: now also IC2G$1.IN4; no longer IC1''.IN6
- net DIO8: no longer IC1''.IN7
- net DIO9: no longer R36.2
- net GND: now also IC1G$1.GND1/2, IC1G$1.GND3/4, IC3G$1.GND1/2, IC3G$1.GND3/4; no longer IC1''.GND, Q11.E, Q13.E, Q9.E, U$23.E
- net IMD_OUT: now also IC3G$1.OUT3; no longer IC1''.OUT6, IC1''.OUT6@2
- net N$11: now also F1.2, SHTDWN_CONN.3; no longer R24.1, U$3.DIO21
- net N$12: now also F2.2, SHTDWN_CONN.2; no longer R25.1, U$3.DIO22
- net N$15: now also F14.2, SHTDWN_CONN.1; no longer D5.A, R8.2, U$3.DIO4
- net N$5: now also U$3.VCC; no longer IC1P1.VBB@4, IC1P1.VBB@5
- net PO1: now also IC1G$1.OUT1; no longer IC1''.OUT1, IC1''.OUT1@2
- net PO2: now also IC1G$1.OUT2; no longer IC1''.OUT2, IC1''.OUT2@2
- net PO3: now also IC1G$1.OUT3; no longer IC1''.OUT3, IC1''.OUT3@2
- net PO4: now also IC1G$1.OUT4; no longer IC1''.OUT4, IC1''.OUT4@2
Other:
- moved on the sheet: BSPD_CONN, D4, F1, F10, F2, F3, F4, F5, F6, F9, R34, R36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

Commit message: more daughter card work
Connections:
- net AI1: now also ACCUMULATOR_CONN.2; no longer ACCUMULATOR_CONN.5
- net AI2: now also ACCUMULATOR_CONN.3; no longer ACCUMULATOR_CONN.6
- net CAN_H: now also ACCUMULATOR_CONN.5; no longer ACCUMULATOR_CONN.3
- net DIO94: now also D6.A, R9.1; no longer D5.A, R8.2
- net DIO95: now also D5.A, R8.2; no longer D6.A, R9.1
- net SHIELD: now also ACCUMULATOR_CONN.6; no longer ACCUMULATOR_CONN.2
