File: EAGLE Models/sbRIO Daughter Card v5/Daughter Card Schematic v5.sch (EAGLE design)
At the start: 70 parts, among them IC1 BTS716G, IC2 BTS716G, IC3 BTS716G, Q7 MMBT4403-7-F, Q8 MMBT4403-7-F, U2 ADXL345, U3 L3G4200D, X1 5566-2

Commit message: Added values for fuses
also rerouted a trace which was unnecesarily long
Parts:
- F1, F14, F2, F6, F7, F8: value (none) -> 0.25A PTC
- F10, F16: value (none) -> 0.5A PTC
- F15, F20, F21, F22: value (none) -> 0.01A PTC
- F17, F18, F19, F9: value (none) -> 1A PTC
- F3, F4, F5: value (none) -> 1mA PTC
Changed lines of the file:
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@@
 <part name="R8" library="resistor" deviceset="R-US_" device="R0402" value="10k"/>
 <part name="R9" library="resistor" deviceset="R-US_" device="R0402" value="10k"/>
-<part name="F3" library="resistor" deviceset="R-EU_" device="R0402"/>
-<part name="F4" library="resistor" deviceset="R-EU_" device="R0402"/>
-<part name="F5" library="resistor" deviceset="R-EU_" device="R0402"/>
-<part name="F6" library="resistor" deviceset="R-EU_" device="R0402"/>
-<part name="F7" library="resistor" deviceset="R-EU_" device="R0402"/>
-<part name="F8" library="resistor" deviceset="R-EU_" device="R0402"/>
-<part name="F16" library="resistor" deviceset="R-EU_" device="R0402"/>
-<part name="F17" library="resistor" deviceset="R-EU_" device="R0402"/>
+<part name="F3" library="resistor" deviceset="R-EU_" device="R0402" value="1mA PTC"/>
+<part name="F4" library="resistor" deviceset="R-EU_" device="R0402" value="1mA PTC"/>
+<part name="F5" library="resistor" deviceset="R-EU_" device="R0402" value="1mA PTC"/>
+<part name="F6" library="resistor" deviceset="R-EU_" device="R0402" value="0.25A PTC"/>
+<part name="F7" library="resistor" deviceset="R-EU_" device="R0402" value="0.25A PTC"/>
+<part name="F8" library="resistor" deviceset="R-EU_" device="R0402" value="0.25A PTC"/>
+<part name="F16" library="resistor" deviceset="R-EU_" device="R0402" value="0.5A PTC"/>
+<part name="F17" library="resistor" deviceset="R-EU_" device="R0402" value="1A PTC"/>
 <part name="Q7" library="formula electric" deviceset="MMBT4403-7-F" device=""/>
 <part name="Q8" library="formula electric" deviceset="MMBT4403-7-F" device=""/>
-<part name="F18" library="resistor" deviceset="R-EU_" device="R0402"/>
+<part name="F18" library="resistor" deviceset="R-EU_" device="R0402" value="1A PTC"/>
 <part name="R13" library="resistor" deviceset="R-US_" device="R0402" value="10k"/>
 <part name="R14" library="resistor" deviceset="R-US_" device="R0402" value="10k"/>
@@
 <part name="R17" library="resistor" deviceset="R-US_" device="R0402" value="10k"/>
 <part name="ACCUMULATOR_CONN" library="con-tycoelectronics" deviceset="RJ45*2" device="1-S" technology="-6L"/>
-<part name="F19" library="resistor" deviceset="R-EU_" device="R0402"/>
+<part name="F19" library="resistor" deviceset="R-EU_" device="R0402" value="1A PTC"/>
 <part name="AIO_PO_CONN" library="con-3m" deviceset="2516-" device="5"/>
-<part name="F15" library="resistor" deviceset="R-EU_" device="R0402"/>
-<part name="F20" library="resistor" deviceset="R-EU_" device="R0402"/>
-<part name="F21" library="resistor" deviceset="R-EU_" device="R0402"/>
-<part name="F22" library="resistor" deviceset="R-EU_" device="R0402"/>
+<part name="F15" library="resistor" deviceset="R-EU_" device="R0402" value="0.01A PTC"/>
+<part name="F20" library="resistor" deviceset="R-EU_" device="R0402" value="0.01A PTC"/>
+<part name="F21" library="resistor" deviceset="R-EU_" device="R0402" value="0.01A PTC"/>
+<part name="F22" library="resistor" deviceset="R-EU_" device="R0402" value="0.01A PTC"/>
 <part name="TUB_CONN" library="con-3m" deviceset="2516-" device="5"/>
 <part name="IC2" library="infineon" deviceset="BTS716G" device=""/>
 <part name="IC1" library="infineon" deviceset="BTS716G" device=""/>
 <part name="IC3" library="infineon" deviceset="BTS716G" device=""/>
-<part name="F1" library="resistor" deviceset="R-EU_" device="R0402"/>
-<part name="F2" library="resistor" deviceset="R-EU_" device="R0402"/>
-<part name="F14" library="resistor" deviceset="R-EU_" device="R0402"/>
-<part name="F9" library="resistor" deviceset="R-EU_" device="R0402"/>
-<part name="F10" library="resistor" deviceset="R-EU_" device="R0402"/>
+<part name="F1" library="resistor" deviceset="R-EU_" device="R0402" value="0.25A PTC"/>
+<part name="F2" library="resistor" deviceset="R-EU_" device="R0402" value="0.25A PTC"/>
+<part name="F14" library="resistor" deviceset="R-EU_" device="R0402" value="0.25A PTC"/>
+<part name="F9" library="resistor" deviceset="R-EU_" device="R0402" value="1A PTC"/>
+<part name="F10" library="resistor" deviceset="R-EU_" device="R0402" value="0.5A PTC"/>
 <part name="X1" library="con-molex" deviceset="5566-2" device=""/>
 <part name="U1" library="SparkFun-DigitalIC" deviceset="TXB0104PWR" device=""/>

Commit message: PTC fuses dont exisist in 0402, made all fuses 0603 instead
Parts:
- F1, F10, F14, F15, F16, F17, F18, F19, F2, F20, F21, F22, F3, F4, F5, F6, F7, F8, F9: device resistor:R-EU_R0402 -> resistor:R-EU_R0603
Changed lines of the file:
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@@
 <grid distance="0.1" unitdist="inch" unit="inch" style="lines" multiple="1" display="no" altdistance="0.01" altunitdist="inch" altunit="inch"/>
 <layers>
-<layer number="1" name="Top" color="1" fill="1" visible="no" active="no"/>
-<layer number="16" name="Bottom" color="4" fill="1" visible="no" active="no"/>
-<layer number="17" name="Pads" color="2" fill="1" visible="no" active="no"/>
-<layer number="18" name="Vias" color="2" fill="1" visible="no" active="no"/>
-<layer number="19" name="Unrouted" color="6" fill="1" visible="no" active="no"/>
-<layer number="20" name="Dimension" color="15" fill="1" visible="no" active="no"/>
-<layer number="21" name="tPlace" color="7" fill="1" visible="no" active="no"/>
-<layer number="22" name="bPlace" color="7" fill="1" visible="no" active="no"/>
-<layer number="23" name="tOrigins" color="15" fill="1" visible="no" active="no"/>
-<layer number="24" name="bOrigins" color="15" fill="1" visible="no" active="no"/>
-<layer number="25" name="tNames" color="7" fill="1" visible="no" active="no"/>
-<layer number="26" name="bNames" color="7" fill="1" visible="no" active="no"/>
-<layer number="27" name="tValues" color="7" fill="1" visible="no" active="no"/>
-<layer number="28" name="bValues" color="7" fill="1" visible="no" active="no"/>
+<layer number="1" name="Top" color="1" fill="1" visible="yes" active="no"/>
+<layer number="16" name="Bottom" color="4" fill="1" visible="yes" active="no"/>
+<layer number="17" name="Pads" color="2" fill="1" visible="yes" active="no"/>
+<layer number="18" name="Vias" color="2" fill="1" visible="yes" active="no"/>
+<layer number="19" name="Unrouted" color="6" fill="1" visible="yes" active="no"/>
+<layer number="20" name="Dimension" color="15" fill="1" visible="yes" active="no"/>
+<layer number="21" name="tPlace" color="7" fill="1" visible="yes" active="no"/>
+<layer number="22" name="bPlace" color="7" fill="1" visible="yes" active="no"/>
+<layer number="23" name="tOrigins" color="15" fill="1" visible="yes" active="no"/>
+<layer number="24" name="bOrigins" color="15" fill="1" visible="yes" active="no"/>
+<layer number="25" name="tNames" color="7" fill="1" visible="yes" active="no"/>
+<layer number="26" name="bNames" color="7" fill="1" visible="yes" active="no"/>
+<layer number="27" name="tValues" color="7" fill="1" visible="yes" active="no"/>
+<layer number="28" name="bValues" color="7" fill="1" visible="yes" active="no"/>
 <layer number="29" name="tStop" color="7" fill="3" visible="no" active="no"/>
 <layer number="30" name="bStop" color="7" fill="6" visible="no" active="no"/>
@@
 <layer number="35" name="tGlue" color="7" fill="4" visible="no" active="no"/>
 <layer number="36" name="bGlue" color="7" fill="5" visible="no" active="no"/>
-<layer number="37" name="tTest" color="7" fill="1" visible="no" active="no"/>
-<layer number="38" name="bTest" color="7" fill="1" visible="no" active="no"/>
+<layer number="37" name="tTest" color="7" fill="1" visible="yes" active="no"/>
+<layer number="38" name="bTest" color="7" fill="1" visible="yes" active="no"/>
 <layer number="39" name="tKeepout" color="4" fill="11" visible="no" active="no"/>
 <layer number="40" name="bKeepout" color="1" fill="11" visible="no" active="no"/>
@@
 <layer number="44" name="Drills" color="7" fill="1" visible="no" active="no"/>
 <layer number="45" name="Holes" color="7" fill="1" visible="no" active="no"/>
-<layer number="46" name="Milling" color="3" fill="1" visible="no" active="no"/>
-<layer number="47" name="Measures" color="7" fill="1" visible="no" active="no"/>
-<layer number="48" name="Document" color="7" fill="1" visible="no" active="no"/>
-<layer number="49" name="Reference" color="7" fill="1" visible="no" active="no"/>
-<layer number="50" name="dxf" color="7" fill="1" visible="no" active="no"/>
-<layer number="51" name="tDocu" color="7" fill="1" visible="no" active="no"/>
-<layer number="52" name="bDocu" color="7" fill="1" visible="no" active="no"/>
-<layer number="53" name="tGND_GNDA" color="7" fill="9" visible="no" active="no"/>
-<layer number="54" name="bGND_GNDA" color="1" fill="9" visible="no" active="no"/>
-<layer number="56" name="wert" color="7" fill="1" visible="no" active="no"/>
+<layer number="46" name="Milling" color="3" fill="1" visible="yes" active="no"/>
+<layer number="47" name="Measures" color="7" fill="1" visible="yes" active="no"/>
+<layer number="48" name="Document" color="7" fill="1" visible="yes" active="no"/>
+<layer number="49" name="Reference" color="7" fill="1" visible="yes" active="no"/>
+<layer number="50" name="dxf" color="7" fill="1" visible="yes" active="no"/>
+<layer number="51" name="tDocu" color="7" fill="1" visible="yes" active="no"/>
+<layer number="52" name="bDocu" color="7" fill="1" visible="yes" active="no"/>
+<layer number="53" name="tGND_GNDA" color="7" fill="9" visible="yes" active="no"/>
+<layer number="54" name="bGND_GNDA" color="1" fill="9" visible="yes" active="no"/>
+<layer number="56" name="wert" color="7" fill="1" visible="yes" active="no"/>
 <layer number="91" name="Nets" color="2" fill="1" visible="yes" active="yes"/>
 <layer number="92" name="Busses" color="1" fill="1" visible="yes" active="yes"/>
@@
 <part name="R8" library="resistor" deviceset="R-US_" device="R0402" value="10k"/>
 <part name="R9" library="resistor" deviceset="R-US_" device="R0402" value="10k"/>
-<part name="F3" library="resistor" deviceset="R-EU_" device="R0402" value="1mA PTC"/>
-<part name="F4" library="resistor" deviceset="R-EU_" device="R0402" value="1mA PTC"/>
-<part name="F5" library="resistor" deviceset="R-EU_" device="R0402" value="1mA PTC"/>
-<part name="F6" library="resistor" deviceset="R-EU_" device="R0402" value="0.25A PTC"/>
-<part name="F7" library="resistor" deviceset="R-EU_" device="R0402" value="0.25A PTC"/>
-<part name="F8" library="resistor" deviceset="R-EU_" device="R0402" value="0.25A PTC"/>
-<part name="F16" library="resistor" deviceset="R-EU_" device="R0402" value="0.5A PTC"/>
-<part name="F17" library="resistor" deviceset="R-EU_" device="R0402" value="1A PTC"/>
+<part name="F3" library="resistor" deviceset="R-EU_" device="R0603" value="1mA PTC"/>
+<part name="F4" library="resistor" deviceset="R-EU_" device="R0603" value="1mA PTC"/>
+<part name="F5" library="resistor" deviceset="R-EU_" device="R0603" value="1mA PTC"/>
+<part name="F6" library="resistor" deviceset="R-EU_" device="R0603" value="0.25A PTC"/>
+<part name="F7" library="resistor" deviceset="R-EU_" device="R0603" value="0.25A PTC"/>
+<part name="F8" library="resistor" deviceset="R-EU_" device="R0603" value="0.25A PTC"/>
+<part name="F16" library="resistor" deviceset="R-EU_" device="R0603" value="0.5A PTC"/>
+<part name="F17" library="resistor" deviceset="R-EU_" device="R0603" value="1A PTC"/>
 <part name="Q7" library="formula electric" deviceset="MMBT4403-7-F" device=""/>
 <part name="Q8" library="formula electric" deviceset="MMBT4403-7-F" device=""/>
-<part name="F18" library="resistor" deviceset="R-EU_" device="R0402" value="1A PTC"/>
+<part name="F18" library="resistor" deviceset="R-EU_" device="R0603" value="1A PTC"/>
 <part name="R13" library="resistor" deviceset="R-US_" device="R0402" value="10k"/>
 <part name="R14" library="resistor" deviceset="R-US_" device="R0402" value="10k"/>
@@
 <part name="R17" library="resistor" deviceset="R-US_" device="R0402" value="10k"/>
 <part name="ACCUMULATOR_CONN" library="con-tycoelectronics" deviceset="RJ45*2" device="1-S" technology="-6L"/>
-<part name="F19" library="resistor" deviceset="R-EU_" device="R0402" value="1A PTC"/>
+<part name="F19" library="resistor" deviceset="R-EU_" device="R0603" value="1A PTC"/>
 <part name="AIO_PO_CONN" library="con-3m" deviceset="2516-" device="5"/>
-<part name="F15" library="resistor" deviceset="R-EU_" device="R0402" value="0.01A PTC"/>
-<part name="F20" library="resistor" deviceset="R-EU_" device="R0402" value="0.01A PTC"/>
-<part name="F21" library="resistor" deviceset="R-EU_" device="R0402" value="0.01A PTC"/>
-<part name="F22" library="resistor" deviceset="R-EU_" device="R0402" value="0.01A PTC"/>
+<part name="F15" library="resistor" deviceset="R-EU_" device="R0603" value="0.01A PTC"/>
+<part name="F20" library="resistor" deviceset="R-EU_" device="R0603" value="0.01A PTC"/>
+<part name="F21" library="resistor" deviceset="R-EU_" device="R0603" value="0.01A PTC"/>
+<part name="F22" library="resistor" deviceset="R-EU_" device="R0603" value="0.01A PTC"/>
 <part name="TUB_CONN" library="con-3m" deviceset="2516-" device="5"/>
 <part name="IC2" library="infineon" deviceset="BTS716G" device=""/>
 <part name="IC1" library="infineon" deviceset="BTS716G" device=""/>
 <part name="IC3" library="infineon" deviceset="BTS716G" device=""/>
-<part name="F1" library="resistor" deviceset="R-EU_" device="R0402" value="0.25A PTC"/>
-<part name="F2" library="resistor" deviceset="R-EU_" device="R0402" value="0.25A PTC"/>
-<part name="F14" library="resistor" deviceset="R-EU_" device="R0402" value="0.25A PTC"/>
-<part name="F9" library="resistor" deviceset="R-EU_" device="R0402" value="1A PTC"/>
-<part name="F10" library="resistor" deviceset="R-EU_" device="R0402" value="0.5A PTC"/>
+<part name="F1" library="resistor" deviceset="R-EU_" device="R0603" value="0.25A PTC"/>
+<part name="F2" library="resistor" deviceset="R-EU_" device="R0603" value="0.25A PTC"/>
+<part name="F14" library="resistor" deviceset="R-EU_" device="R0603" value="0.25A PTC"/>
+<part name="F9" library="resistor" deviceset="R-EU_" device="R0603" value="1A PTC"/>
+<part name="F10" library="resistor" deviceset="R-EU_" device="R0603" value="0.5A PTC"/>
 <part name="X1" library="con-molex" deviceset="5566-2" device=""/>
 <part name="U1" library="SparkFun-DigitalIC" deviceset="TXB0104PWR" device=""/>

Commit message: some of the 0603 PTC fuses were not possible to lay on board well
replaced with normal fuses
Parts:
- F15, F20, F21, F22: device resistor:R-EU_R0603 -> resistor:R-EU_R0402
Changed lines of the file:
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@@
 <part name="F19" library="resistor" deviceset="R-EU_" device="R0603" value="1A PTC"/>
 <part name="AIO_PO_CONN" library="con-3m" deviceset="2516-" device="5"/>
-<part name="F15" library="resistor" deviceset="R-EU_" device="R0603" value="0.01A PTC"/>
-<part name="F20" library="resistor" deviceset="R-EU_" device="R0603" value="0.01A PTC"/>
-<part name="F21" library="resistor" deviceset="R-EU_" device="R0603" value="0.01A PTC"/>
-<part name="F22" library="resistor" deviceset="R-EU_" device="R0603" value="0.01A PTC"/>
+<part name="F15" library="resistor" deviceset="R-EU_" device="R0402" value="0.01A PTC"/>
+<part name="F20" library="resistor" deviceset="R-EU_" device="R0402" value="0.01A PTC"/>
+<part name="F21" library="resistor" deviceset="R-EU_" device="R0402" value="0.01A PTC"/>
+<part name="F22" library="resistor" deviceset="R-EU_" device="R0402" value="0.01A PTC"/>
 <part name="TUB_CONN" library="con-3m" deviceset="2516-" device="5"/>
 <part name="IC2" library="infineon" deviceset="BTS716G" device=""/>

Commit message: changed step-down diodes into linear regulators
also made schematic far more readable, and removed some unnecessary
outputs on TUB_CONN
Parts:
- removed D1, D2, D4, D5, D6: MMBZ5238B-7-F, formula electric:MMBZ5238B-7-F
- removed F10: 0.5A PTC, resistor:R-EU_R0603
- removed F7, F8: 0.25A PTC, resistor:R-EU_R0603
- removed F9: 1A PTC, resistor:R-EU_R0603
- removed R14, R17, R34, R8, R9: 10k, resistor:R-US_R0402
- removed X2: (no value), con-amp:FTOP-4
- added C16, C17, C18, C19, C20: 1uF, SparkFun-Passives:CAP0603-CAP
- added R1, R2, R3, R4, R5: 10k, resistor:R-US_R0402
- added U$1, U$4, U$5, U$6, U$7: MIC5225-3.3YM5-TR, formula electric:MIC5225-3.3YM5-TR
- added WHEEL: (no value), con-amp:FTOP-4
Connections:
- net AI3 renamed BRAKE_PRESS_IN_1
- net AI4 renamed BRAKE_PRESS_IN_2
- net BSPD5 renamed THROTTLE_OK_OUT
- net PO1 renamed ACCUMULATOR_FANS
- net THROTTLE_1 renamed THROTTLE_IN_1
- net THROTTLE_2 renamed THROTTLE_IN_2
- removed net AMS_OK: D6.C, F8.2
- removed net IMD_OK: D5.C, F7.2
- removed net N$1: D2.C, SBRIO_AUX.LATCH
- removed net N$13: ACCUMULATOR_CONN.7, F8.1
- removed net N$14: ACCUMULATOR_CONN.8, F7.1
- removed net N$16: F9.1, TUB_CONN-3.KL
- removed net N$17: F10.1, TUB_CONN-1.KL
- removed net N$2: D1.C, SBRIO_AUX.E-STOP
- removed net N$42: BSPD_CONN.1, D4.C
- removed net N$55: F17.1, SBRIO_AUX.POS_AIR
- removed net N$59: F18.1, SBRIO_AUX.DIO39
- new net 5V_IO_1: F17.1
- new net AMS_OK_IN: ACCUMULATOR_CONN.7, R1.1, U$4.3~16V_IN
- new net BSPD_OK_IN: BSPD_CONN.1, R2.1, U$5.3~16V_IN
- new net DC_DC_DISABLE: F18.1
- new net E-STOP_OK: R3.1, U$6.3~16V_IN
- new net IMD_OK_IN: ACCUMULATOR_CONN.8, R5.1, U$1.3~16V_IN
- new net LATCH_OK: R4.1, U$7.3~16V_IN
- net 12V: no longer F9.2
- net 5V: no longer F10.2
- net CAN_GND: now also TUB_CONN-10.KL
- net DIO1: now also C16.1, U$7.3.3V_OUT; no longer D4.A, R34.2
- net DIO13: now also C17.1, U$6.3.3V_OUT; no longer D1.A, R17.1
- net DIO14: now also C18.1, U$5.3.3V_OUT; no longer D2.A, R14.1
- net DIO94: now also C19.1, U$4.3.3V_OUT; no longer D6.A, R9.1
- net DIO95: now also C20.1, U$1.3.3V_OUT; no longer D5.A, R8.2
- net GND: now also C16.2, C17.2, C18.2, C19.2, C20.2, R1.2, R2.2, R3.2, R4.2, R5.2, U$1.GND, U$4.GND, U$5.GND, U$6.GND, U$7.GND; no longer R14.2, R17.2, R34.1, R8.1, R9.2, TUB_CONN-10.KL
- net WS1: now also WHEEL-1.1; no longer X2-1.1
- net WS2: now also WHEEL-2.1; no longer X2-2.1
- net WS3: now also WHEEL-3.1; no longer X2-3.1
- net WS4: now also WHEEL-4.1; no longer X2-4.1
Other:
- note added: "12V high side drivers"
- note added: "3.3V and 5V Voltage Regulators"
- note added: "Accelerometer"
- note added: "Amplified 5V Outputs"
- note added: "Auxiliary ribbon cable connector"
- note added: "Connectors for tub and accumulator outputs"
- note added: "Gyroscope"
- note added: "Shutdown and BSPD Clamp Connectors"
- note added: "Wheel Speed input connector and Level Shifter"
- note added: "pull down resistor"
- note added: "sbRIO CAN ribbon connector"
- note added: "sbRIO mezzanine connector"
- note added: "sbRIO_J502 Auxiliary ribbon connector"
- note added: "step down 12V+5V inputs to 3.3V"
- note removed: "need fusing"
- moved on the sheet: 3.3V_REG, 5V_REG, ACCUMULATOR_CONN, AIO_PO_CONN-1, AIO_PO_CONN-10, AIO_PO_CONN-11, AIO_PO_CONN-12, AIO_PO_CONN-13, AIO_PO_CONN-14, AIO_PO_CONN-15, AIO_PO_CONN-16, AIO_PO_CONN-2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
