File: EAGLE Models/Dashboard/Dashboard.sch (EAGLE design)
At the start: 86 parts, among them IC1 AT90CAN128, IC2 MCP2551SO8, IC3 NUP2105L, IC5 FT232RL, Q1 56P2859, U1 74LCX125M

Commit message: Merge Combustion EAGLE documents and cleanup some of the repo.
Parts:
- removed 12V_PWR: M01PTH, SparkFun-Connectors:M01PTH
- removed CAN_UC_CONN, DRIVER_OUTPUTS: (no value), SparkFun-Connectors:M081X08
- removed DRIVER_INPUTS_1, DRIVER_INPUTS_3: (no value), SparkFun-Connectors:M05PTH
- removed DRIVER_INPUTS_2: (no value), SparkFun-Connectors:M03PTH
- added CANPWR, LEDOUT: MICRO5LOCK, DashAndCAN library:MICRO5LOCK
- added ROT/PUSH: MICRO6LOCK, DashAndCAN library:MICRO6LOCK
- added U$14: MUSBB, DashAndCAN library:MUSBB
Connections:
- removed net AVR_SCK: IC1.(SCK)PB1
- net 12V: now also CANPWR.P$2; no longer 12V_PWR.1
- net AVR_SCLK: now also IC1.(SCK)PB1
- net CAN_H: now also CANPWR.P$4; no longer CAN_UC_CONN.4
- net CAN_L: now also CANPWR.P$3; no longer CAN_UC_CONN.3
- net D+: now also U$14.P$3; no longer CAN_UC_CONN.6
- net D-: now also U$14.P$2; no longer CAN_UC_CONN.7
- net DRV1: now also LEDOUT.P$2; no longer DRIVER_OUTPUTS.2
- net DRV2: now also LEDOUT.P$3; no longer DRIVER_OUTPUTS.3
- net DRV3: now also LEDOUT.P$4; no longer DRIVER_OUTPUTS.4
- net DRV4: no longer DRIVER_OUTPUTS.5
- net GND: now also CANPWR.P$1, LEDOUT.P$1, ROT/PUSH.P$4, U$14.P$5; no longer CAN_UC_CONN.2, CAN_UC_CONN.5, DRIVER_OUTPUTS.8
- net PA0: no longer DRIVER_OUTPUTS.6
- net PA1: no longer DRIVER_OUTPUTS.7
- net PA7: no longer DRIVER_INPUTS_3.1
- net PC0: now also ROT/PUSH.P$1; no longer DRIVER_INPUTS_1.1
- net PC1: no longer DRIVER_INPUTS_1.2
- net PC2: no longer DRIVER_INPUTS_1.3
- net PC3: no longer DRIVER_INPUTS_1.4
- net PC4: no longer DRIVER_INPUTS_1.5
- net PC5: no longer DRIVER_INPUTS_3.5
- net PC6: no longer DRIVER_INPUTS_3.4
- net PC7: no longer DRIVER_INPUTS_3.3
- net PF0: now also ROT/PUSH.P$5; no longer DRIVER_INPUTS_2.1
- net PF1: now also ROT/PUSH.P$3; no longer DRIVER_INPUTS_2.2
- net PF2: now also ROT/PUSH.P$2; no longer DRIVER_INPUTS_2.3
- net PG2: no longer DRIVER_INPUTS_3.2
- net USB_V_IN: now also U$14.P$1; no longer CAN_UC_CONN.8
- net VCC: now also CANPWR.P$5, ROT/PUSH.P$6; no longer CAN_UC_CONN.1, DRIVER_OUTPUTS.1
Other:
- note added: "potentiometer"
- note added: "push/flag"
