File: EAGLE Models/Accel Gyro GPS Module/Accel Gyro GPS Module.sch (EAGLE design)
At the start: 71 parts, among them IC1 AT90CAN128, IC2 MCP2551SO8, IC3 NUP2105L, IC5 FT232RL, Q1 56P2859, U1 74LCX125M, U2 MPU-6000QFN-24, U3 74LCX125M

Commit message: More repository cleanup.
Parts:
- removed 12V_PWR: M01PTH, SparkFun-Connectors:M01PTH
- removed C5: 2.2nF, SparkFun-Capacitors:2.2NF/2200PF-50V-10%(0603)
- removed C6, C7: 0.1uF, SparkFun-Capacitors:.1UF-CERCAP-08604
- removed CAN_UC_CONN, DRIVER_OUTPUTS: (no value), SparkFun-Connectors:M081X08
- removed DRIVER_INPUTS_1, DRIVER_INPUTS_3: (no value), SparkFun-Connectors:M05PTH
- removed DRIVER_INPUTS_2: (no value), SparkFun-Connectors:M03PTH
- removed F2, F3, F4, F5: 15V,0.5A, SparkFun:PTCSMD
- removed R11, R12, R13, R14, R15, R16, R4, R5: (no value), SparkFun-Resistors:RESISTOR0603
- removed SJ2, SJ3: (no value), jumper:SJ2W
- removed SJ4: (no value), jumper:SJ
- removed U$10, U$12, U$6, U$8: MMBT4403-7-F, formula electric:MMBT4403-7-F
- removed U$11, U$5, U$7, U$9: MMBT4401-7-F, formula electric:MMBT4401-7-F
- removed U1, U3: 74LCX125M, Fairchild_By_element14_Batch_1:74LCX125M
- removed U2: MPU-6000QFN-24, SparkFun-Sensors:MPU-6000QFN-24
- added CANPWR: MICRO5LOCK, DashAndCAN library:MICRO5LOCK
- added ROT/PUSH: MICRO6LOCK, DashAndCAN library:MICRO6LOCK
- added U$14: MUSBB, DashAndCAN library:MUSBB
Connections:
- removed net AVR_SCK: H7.3, IC1.(SCK)PB1, SJ3.3, U1.A3
- removed net AVR_SPI_IN: SJ4.2, U3.O2
- removed net AVR_SPI_OUT: SJ2.2, U3.O1
- removed net AVR_SPI_SS1: U3.O3
- removed net DRV1: DRIVER_OUTPUTS.2, F5.2
- removed net DRV2: DRIVER_OUTPUTS.3, F4.2
- removed net DRV3: DRIVER_OUTPUTS.4, F3.2
- removed net DRV4: DRIVER_OUTPUTS.5, F2.2
- removed net FT801_CS_N: U1.O0
- removed net FT801_MISO: U1.A1
- removed net FT801_MOSI: U1.O2
- removed net FT801_SCLK: U1.O3
- removed net MPU_SCL: U2.SCL/SCLK, U3.A0
- removed net MPU_SD0: U2.AD0/SDO, U3.A2
- removed net MPU_SDI: U2.SDA/SDI, U3.A1
- removed net MPU_SPI_SS: U2.CS, U3.A3
- removed net N$1: U1.GND, U3.GND
- removed net N$2: IC1.(SDA/INT1)PD1, SJ2.1
- removed net N$23: R5.2, U$5.B
- removed net N$24: R4.2, U$6.B
- removed net N$25: R4.1, U$5.C
- removed net N$26: F2.1, U$6.C
- removed net N$27: R12.2, U$7.B
- removed net N$28: R11.2, U$8.B
- removed net N$29: R11.1, U$7.C
- removed net N$3: IC1.(SCL/INT0)PD0, SJ3.1
- removed net N$30: F3.1, U$8.C
- removed net N$31: R14.2, U$9.B
- removed net N$33: R13.2, U$10.B
- removed net N$37: R13.1, U$9.C
- removed net N$38: F4.1, U$10.C
- removed net N$39: R16.2, U$11.B
- removed net N$4: C6.2, U2.REGOUT
- removed net N$40: R15.2, U$12.B
- removed net N$41: R15.1, U$11.C
- removed net N$42: F5.1, U$12.C
- removed net N$7: C5.2, U2.CPOUT
- new net SCL: IC1.(SCL/INT0)PD0
- new net SDA: IC1.(SDA/INT1)PD1
- net 12V: now also CANPWR.P$2; no longer 12V_PWR.1
- net 12V_PROTECTED: no longer U$10.E, U$12.E, U$6.E, U$8.E
- net 3.3V: no longer C7.1, U1.VCC, U2.VDD, U3.VCC
- net AVR_CS: no longer U1.A0
- net AVR_MISO: no longer U1.O1
- net AVR_MOSI: no longer SJ2.3, U1.A2
- net AVR_SCLK: now also H7.3, IC1.(SCK)PB1; no longer SJ3.2, U3.O0
- net CAN_H: now also CANPWR.P$4; no longer CAN_UC_CONN.4
- net CAN_L: now also CANPWR.P$3; no longer CAN_UC_CONN.3
- net D+: now also U$14.P$3; no longer CAN_UC_CONN.6
- net D-: now also U$14.P$2; no longer CAN_UC_CONN.7
- net GND: now also CANPWR.P$1, ROT/PUSH.P$4, U$14.P$5; no longer C5.1, C6.1, C7.2, CAN_UC_CONN.2, CAN_UC_CONN.5, DRIVER_OUTPUTS.8, U$11.E, U$5.E, U$7.E, U$9.E, U1.~OE0, U1.~OE1, U1.~OE2, U1.~OE3, U2.CLKIN, U2.FSYNC, U2.GND, U3.~OE0, U3.~OE1, U3.~OE2, U3.~OE3
- net PA0: no longer DRIVER_OUTPUTS.6
- net PA1: no longer DRIVER_OUTPUTS.7
- net PA7: no longer DRIVER_INPUTS_3.1
- net PB4(PWM): no longer R5.1
- net PB5(PWM): no longer R12.1
- net PB6(PWM): no longer R14.1
- net PB7(PWM): no longer R16.1
- net PC0: now also ROT/PUSH.P$1; no longer DRIVER_INPUTS_1.1
- net PC1: no longer DRIVER_INPUTS_1.2
- net PC2: no longer DRIVER_INPUTS_1.3
- net PC3: no longer DRIVER_INPUTS_1.4
- net PC4: no longer DRIVER_INPUTS_1.5
- net PC5: no longer DRIVER_INPUTS_3.5
- net PC6: no longer DRIVER_INPUTS_3.4
- net PC7: no longer DRIVER_INPUTS_3.3
- net PF0: now also ROT/PUSH.P$5; no longer DRIVER_INPUTS_2.1
- net PF1: now also ROT/PUSH.P$3; no longer DRIVER_INPUTS_2.2
- net PF2: now also ROT/PUSH.P$2; no longer DRIVER_INPUTS_2.3
- net PG2: no longer DRIVER_INPUTS_3.2
- net RESET: no longer U2.INT
- net USB_V_IN: now also U$14.P$1; no longer CAN_UC_CONN.8
- net VCC: now also CANPWR.P$5, ROT/PUSH.P$6; no longer CAN_UC_CONN.1, DRIVER_OUTPUTS.1
Other:
- note added: "Connectors/Headers"
- note added: "potentiometer"
- note added: "push/flag"
- note removed: "GPS_MODULE(3.3v)<->AVR(5.0V) Level Shifter"
- note removed: "Headers"
- note removed: "High-Side Drivers"
- note removed: "Invensense MPU 6000 Accelerometer and Gyroscope(SPI or I2C)"
- note removed: "MPU(3.3v)<->AVR(5.0V) Level Shifter"
- moved on the sheet: C1, C12, C13, C14, C15, C16, C18, C19, C2, C20, C3, C4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
